File: pcb/FiveChannel/Channels.kicad_sch (KiCad schematic)
At the start: 11 parts, among them J201 Conn_01x20_Male

Commit message: Updates the schematic and PCB design to the lastest from the original repo
Parts:
- renumbered J201 to J?, R201 to R?, R202 to R?, R203 to R?, R204 to R?, R205 to R?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
